File: PCB/ROVPCB/ROVPCB.kicad_pcb (KiCad board)
At the start: 2 copper layers, 65 x 56 mm, 15 parts, among them J1 Conn_01x04_Male, J2 Conn_01x04_Male, P1 Conn_02x20_Odd_Even, U1 MPU-9250, U2 BME280, U3 LIGHT_TSL2591, U4 LTC4316IDDPBF

Commit message: Adding the Atlas Board... BNC??
Parts:
- added U5: AtlasOEM, Adafruit TSL2591:OEM Board, F.Cu at (237.0, 136.7)
Connections:
- U2 pad 3: /GPIO2(SDA1) -> Net-(U2-Pad3)
- U2 pad 4: /GPIO3(SCL1) -> Net-(U2-Pad4)
- U4 pad 1: Net-(U4-Pad1) -> GND
- U4 pad 10: Net-(U4-Pad10) -> /GPIO3(SCL1)
- U4 pad 11: Net-(U4-Pad11) -> GND
- U4 pad 2: Net-(U4-Pad2) -> GND
- U4 pad 3: Net-(U4-Pad3) -> +3V3
- U4 pad 4: Net-(U4-Pad4) -> +3V3
- U4 pad 7: Net-(U4-Pad7) -> /GPIO2(SDA1)
- U4 pad 8: Net-(U4-Pad8) -> Net-(U2-Pad3)
- U4 pad 9: Net-(U4-Pad9) -> Net-(U2-Pad4)
Routing:
- net +3V3: track 52.5 -> 52.6 mm, vias 0 -> 1
Changed lines of the file:
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@@
     (thickness 1.6)
     (drawings 29)
-    (tracks 40)
+    (tracks 44)
     (zones 0)
-    (modules 15)
-    (nets 52)
+    (modules 16)
+    (nets 51)
   )
   (page A3)
@@
   (net 39 "Net-(U3-Pad2)")
   (net 40 "Net-(U3-Pad4)")
-  (net 41 "Net-(U4-Pad1)")
-  (net 42 "Net-(U4-Pad2)")
-  (net 43 "Net-(U4-Pad3)")
-  (net 44 "Net-(U4-Pad4)")
-  (net 45 "Net-(U4-Pad5)")
-  (net 46 "Net-(U4-Pad6)")
-  (net 47 "Net-(U4-Pad7)")
-  (net 48 "Net-(U4-Pad8)")
-  (net 49 "Net-(U4-Pad9)")
-  (net 50 "Net-(U4-Pad10)")
-  (net 51 "Net-(U4-Pad11)")
+  (net 41 "Net-(U4-Pad5)")
+  (net 42 "Net-(U4-Pad6)")
+  (net 43 "Net-(U2-Pad4)")
+  (net 44 "Net-(U2-Pad3)")
+  (net 45 "Net-(U5-Pad2)")
+  (net 46 "Net-(U5-Pad4)")
+  (net 47 "Net-(U5-Pad5)")
+  (net 48 "Net-(U5-Pad7)")
+  (net 49 "Net-(U5-Pad9)")
+  (net 50 "Net-(U5-Pad10)")
   (net_class Default "This is the default net class."
     (clearance 0.2)
@@
     (add_net "Net-(U1-Pad21)")
     (add_net "Net-(U1-Pad7)")
+    (add_net "Net-(U2-Pad3)")
+    (add_net "Net-(U2-Pad4)")
     (add_net "Net-(U3-Pad2)")
     (add_net "Net-(U3-Pad4)")
-    (add_net "Net-(U4-Pad1)")
-    (add_net "Net-(U4-Pad10)")
-    (add_net "Net-(U4-Pad11)")
-    (add_net "Net-(U4-Pad2)")
-    (add_net "Net-(U4-Pad3)")
-    (add_net "Net-(U4-Pad4)")
     (add_net "Net-(U4-Pad5)")
     (add_net "Net-(U4-Pad6)")
-    (add_net "Net-(U4-Pad7)")
-    (add_net "Net-(U4-Pad8)")
-    (add_net "Net-(U4-Pad9)")
+    (add_net "Net-(U5-Pad10)")
+    (add_net "Net-(U5-Pad2)")
+    (add_net "Net-(U5-Pad4)")
+    (add_net "Net-(U5-Pad5)")
+    (add_net "Net-(U5-Pad7)")
+    (add_net "Net-(U5-Pad9)")
   )
   (net_class Power ""
@@
     (fp_line (start 1.41 1.54) (end -1.41 1.54) (layer F.CrtYd) (width 0.05))
     (pad 4 smd rect (at 0.975 -1.025 90) (size 0.5 0.35) (layers F.Cu F.Paste F.Mask)
-      (net 10 "/GPIO3(SCL1)"))
+      (net 43 "Net-(U2-Pad4)"))
     (pad 3 smd rect (at 0.325 -1.025 90) (size 0.5 0.35) (layers F.Cu F.Paste F.Mask)
-      (net 9 "/GPIO2(SDA1)"))
+      (net 44 "Net-(U2-Pad3)"))
     (pad 2 smd rect (at -0.325 -1.025 90) (size 0.5 0.35) (layers F.Cu F.Paste F.Mask)
       (net 1 +3V3))
@@
     (fp_arc (start 0 -1.5494) (end -0.3048 -1.5494) (angle -180) (layer Eco2.User) (width 0.1524))
     (pad 1 smd rect (at -1.4478 -1) (size 0.8128 0.3048) (layers F.Cu F.Paste F.Mask)
-      (net 41 "Net-(U4-Pad1)"))
+      (net 3 GND))
     (pad 2 smd rect (at -1.4478 -0.5) (size 0.8128 0.3048) (layers F.Cu F.Paste F.Mask)
-      (net 42 "Net-(U4-Pad2)"))
+      (net 3 GND))
     (pad 3 smd rect (at -1.4478 0) (size 0.8128 0.3048) (layers F.Cu F.Paste F.Mask)
-      (net 43 "Net-(U4-Pad3)"))
+      (net 1 +3V3))
     (pad 4 smd rect (at -1.4478 0.5) (size 0.8128 0.3048) (layers F.Cu F.Paste F.Mask)
-      (net 44 "Net-(U4-Pad4)"))
+      (net 1 +3V3))
     (pad 5 smd rect (at -1.4478 1) (size 0.8128 0.3048) (layers F.Cu F.Paste F.Mask)
-      (net 45 "Net-(U4-Pad5)"))
+      (net 41 "Net-(U4-Pad5)"))
     (pad 6 smd rect (at 1.4478 1) (size 0.8128 0.3048) (layers F.Cu F.Paste F.Mask)
-      (net 46 "Net-(U4-Pad6)"))
+      (net 42 "Net-(U4-Pad6)"))
     (pad 7 smd rect (at 1.4478 0.5) (size 0.8128 0.3048) (layers F.Cu F.Paste F.Mask)
-      (net 47 "Net-(U4-Pad7)"))
+      (net 9 "/GPIO2(SDA1)"))
     (pad 8 smd rect (at 1.4478 0) (size 0.8128 0.3048) (layers F.Cu F.Paste F.Mask)
-      (net 48 "Net-(U4-Pad8)"))
+      (net 44 "Net-(U2-Pad3)"))
     (pad 9 smd rect (at 1.4478 -0.5) (size 0.8128 0.3048) (layers F.Cu F.Paste F.Mask)
-      (net 49 "Net-(U4-Pad9)"))
+      (net 43 "Net-(U2-Pad4)"))
     (pad 10 smd rect (at 1.4478 -1) (size 0.8128 0.3048) (layers F.Cu F.Paste F.Mask)
-      (net 50 "Net-(U4-Pad10)"))
+      (net 10 "/GPIO3(SCL1)"))
     (pad 11 smd rect (at 0 0) (size 1.7526 2.4892) (layers F.Cu F.Paste F.Mask)
-      (net 51 "Net-(U4-Pad11)"))
+      (net 3 GND))
+  )
+  (module "Adafruit TSL2591:OEM Board" (layer F.Cu)
+    (at 237.01 136.66)
+    (fp_text reference U5 (at 0.05 1.8) (layer F.SilkS)
+      (effects (font (size 1 1) (thickness 0.15)))
+    )
+    (fp_text value AtlasOEM (at 0.05 0.8) (layer F.Fab)
+      (effects (font (size 1 1) (thickness 0.15)))
+    )
+    (fp_line (start 6.05 5.3) (end -5.95 5.3) (layer F.SilkS) (width 0.15))
+    (fp_line (start -5.95 -5.7) (end 6.05 -5.7) (layer F.SilkS) (width 0.15))
+    (pad 10 smd rect (at 6.05 -4.8) (size 2.5 1.4) (layers F.Cu F.Paste F.Mask)
+      (net 50 "Net-(U5-Pad10)"))
+    (pad 9 smd rect (at 6.05 -2.5) (size 2.5 1.4) (layers F.Cu F.Paste F.Mask)
+      (net 49 "Net-(U5-Pad9)"))
+    (pad 8 smd rect (at 6.1 -0.2) (size 2.5 1.4) (layers F.Cu F.Paste F.Mask)
+      (net 10 "/GPIO3(SCL1)"))
+    (pad 7 smd rect (at 6.05 2.1) (size 2.5 1.4) (layers F.Cu F.Paste F.Mask)
+      (net 48 "Net-(U5-Pad7)"))
+    (pad 6 smd rect (at 6.05 4.4) (size 2.5 1.4) (layers F.Cu F.Paste F.Mask)
+      (net 3 GND))
+    (pad 1 smd rect (at -5.85 -4.8) (size 2.5 1.4) (layers F.Cu F.Paste F.Mask)
+      (net 9 "/GPIO2(SDA1)"))
+    (pad 2 smd rect (at -5.85 -2.5) (size 2.5 1.4) (layers F.Cu F.Paste F.Mask)
+      (net 45 "Net-(U5-Pad2)"))
+    (pad 3 smd rect (at -5.85 -0.2) (size 2.5 1.4) (layers F.Cu F.Paste F.Mask)
+      (net 1 +3V3))
+    (pad 4 smd rect (at -5.85 2.1) (size 2.5 1.4) (layers F.Cu F.Paste F.Mask)
+      (net 46 "Net-(U5-Pad4)"))
+    (pad 5 smd rect (at -5.85 4.4) (size 2.5 1.4) (layers F.Cu F.Paste F.Mask)
+      (net 47 "Net-(U5-Pad5)"))
   )
   (gr_line (start 200 112.9795) (end 200 131.0135) (layer Edge.Cuts) (width 0.1))
@@
   (segment (start 208.93 99.33) (end 208.37 98.77) (width 0.2) (layer F.Cu) (net 1))
   (segment (start 208.93 105.55) (end 208.93 99.33) (width 0.2) (layer F.Cu) (net 1))
-  (segment (start 208.93 105.55) (end 208.93 110.63) (width 0.2) (layer F.Cu) (net 1))
   (segment (start 228.69 98.77) (end 228.69 99.972081) (width 0.2) (layer F.Cu) (net 1))
-  (segment (start 215.492081 113.17) (end 208.89 113.17) (width 0.2) (layer F.Cu) (net 1))
-  (segment (start 208.93 113.13) (end 208.93 110.63) (width 0.2) (layer F.Cu) (net 1))
   (segment (start 208.89 113.17) (end 208.93 113.13) (width 0.2) (layer F.Cu) (net 1))
   (segment (start 216.51 122.135) (end 216.51 112.152081) (width 0.2) (layer F.Cu) (net 1))
@@
   (segment (start 228.69 99.972081) (end 216.51 112.152081) (width 0.2) (layer F.Cu) (net 1))
   (segment (start 216.51 112.152081) (end 215.492081 113.17) (width 0.2) (layer F.Cu) (net 1))
+  (via (at 209.09 113.17) (size 0.9) (drill 0.6) (layers F.Cu B.Cu) (net 1))
+  (segment (start 208.93 113.01) (end 209.09 113.17) (width 0.2) (layer B.Cu) (net 1))
+  (segment (start 208.93 110.63) (end 208.93 113.01) (width 0.2) (layer B.Cu) (net 1))
+  (segment (start 215.492081 113.17) (end 209.09 113.17) (width 0.2) (layer F.Cu) (net 1))
+  (segment (start 209.09 113.17) (end 208.89 113.17) (width 0.2) (layer F.Cu) (net 1))
+  (segment (start 208.93 105.55) (end 208.93 110.63) (width 0.2) (layer B.Cu) (net 1))
   (segment (start 208.37 96.23) (end 210.91 96.23) (width 0.2) (layer F.Cu) (net 2))
   (via (at 215.24 118.25) (size 0.9) (drill 0.6) (layers F.Cu B.Cu) (net 3))
@@
   (segment (start 210.18 99.5) (end 210.91 98.77) (width 0.2) (layer F.Cu) (net 9))
   (segment (start 210.18 105.55) (end 210.18 99.5) (width 0.2) (layer F.Cu) (net 9))
-  (segment (start 210.18 105.55) (end 210.18 110.63) (width 0.2) (layer F.Cu) (net 9))
   (via (at 210.16 114.44) (size 0.9) (drill 0.6) (layers F.Cu B.Cu) (net 9))
   (segment (start 212.2 119.52) (end 212.2 116.48) (width 0.2) (layer F.Cu) (net 9))
@@
   (segment (start 210.16 110.65) (end 210.18 110.63) (width 0.2) (layer B.Cu) (net 9))
   (segment (start 210.16 114.44) (end 210.16 110.65) (width 0.2) (layer B.Cu) (net 9))
+  (segment (start 210.18 105.55) (end 210.18 110.63) (width 0.2) (layer B.Cu) (net 9))
   (segment (start 211.43 100.79) (end 211.43 105.55) (width 0.2) (layer F.Cu) (net 10))
   (segment (start 213.45 98.77) (end 211.43 100.79) (width 0.2) (layer F.Cu) (net 10))
-  (segment (start 211.43 105.55) (end 211.43 110.63) (width 0.2) (layer F.Cu) (net 10))
   (via (at 211.43 114.44) (size 0.9) (drill 0.6) (layers F.Cu B.Cu) (net 10))
   (segment (start 211.43 110.63) (end 211.43 114.44) (width 0.2) (layer B.Cu) (net 10))
   (segment (start 212.7 115.71) (end 212.7 119.52) (width 0.2) (layer F.Cu) (net 10))
   (segment (start 211.43 114.44) (end 212.7 115.71) (width 0.2) (layer F.Cu) (net 10))
+  (segment (start 211.43 106.45) (end 211.43 110.63) (width 0.2) (layer B.Cu) (net 10))
+  (segment (start 211.43 105.55) (end 211.43 106.45) (width 0.2) (layer B.Cu) (net 10))
   (segment (start 211.43 125.565) (end 212.7 124.295) (width 0.2) (layer F.Cu) (net 33))
   (segment (start 212.7 124.295) (end 212.7 123.42) (width 0.2) (layer F.Cu) (net 33))

Commit message: BNCgit add * Boiz
Parts:
- added J3: Conn_Coaxial, footprints:5227161-1, F.Cu at (209.4, 134.7)
- moved R1 33.2 mm to (211.2, 125.8), turned to 180 degrees
- moved U4 23.8 mm to (233.0, 106.7)
- moved U3 16.1 mm to (226.0, 105.1)
- moved U2 12.9 mm to (232.9, 110.7), turned to 270 degrees
- moved U5 9.47 mm to (228.1, 133.5)
- moved C3 6.91 mm to (218.3, 121.6)
- moved C1 2.50 mm to (213.9, 125.9)
- moved C2 1.76 mm to (216.4, 125.3)
Routing:
- net /GPIO3(SCL1): track 22.1 -> 105.3 mm, vias 1 -> 8
- net +3V3: track 52.6 -> 128.5 mm, vias 1 -> 11
- net /GPIO2(SDA1): track 21.9 -> 89.6 mm, vias 1 -> 6
- net Net-(U2-Pad4): track 0.00 -> 17.4 mm, vias 0 -> 2
- net Net-(J3-Pad1): track 0.00 -> 14.1 mm
- net Net-(J3-Pad2): track 0.00 -> 13.5 mm, vias 0 -> 1
- net Net-(U2-Pad3): track 0.00 -> 8.85 mm, vias 0 -> 2
- net Net-(C2-Pad1): track 3.09 -> 0.00 mm
- net GND: track 3.49 -> 0.50 mm, vias 2 -> 3
- net Net-(R1-Pad1): track 0.00 -> 2.82 mm
- net Net-(C3-Pad1): track 2.64 -> 0.00 mm
- net Net-(C1-Pad1): track 2.67 -> 1.79 mm
Other:
- board text added: "Accel."
- board text added: "Atlas"
- board text added: "Lux"
- board text added: "Pressure"
- board text added: "Temp"
- board text added: "Temp/Press/Humid"
- board text removed: "Sensor1"
- board text removed: "Sensor2"
