File: PCB/ROVPCB/ROVPCB.sch (KiCad schematic (older format))
At the start: 16 parts, among them J1 Conn_01x04_Male, J2 Conn_01x04_Male, P1 Conn_02x20_Odd_Even, U1 MPU-9250, U2 BME280, U3 LIGHT_TSL2591, U4 LTC4316IDDPBF, U5 AtlasOEM

Commit message: BNCgit add * Boiz
Parts:
- added J3: Conn_Coaxial, footprints:5227161-1, symbol Connector:Conn_Coaxial
Connections:
- wire segments 122 -> 125
Other:
- note added: "50 Ohm BNC"
Changed lines of the file:
@@
 	9550 1450 9000 1450
 $Comp
-L ROVPCB-rescue:GND-power-ROVPCB-rescue-ROVPCB-rescue #PWR?
+L ROVPCB-rescue:GND-power-ROVPCB-rescue-ROVPCB-rescue #PWR010
 U 1 1 5CBFDF85
 P 9250 1650
-F 0 "#PWR?" H 9250 1400 50  0001 C CNN
+F 0 "#PWR010" H 9250 1400 50  0001 C CNN
 F 1 "GND" H 9250 1500 50  0000 C CNN
 F 2 "" H 9250 1650 50  0000 C CNN
@@
 	9250 1650 9000 1650
 $Comp
-L ROVPCB-rescue:+3.3V-power-ROVPCB-rescue-ROVPCB-rescue #PWR?
+L ROVPCB-rescue:+3.3V-power-ROVPCB-rescue-ROVPCB-rescue #PWR09
 U 1 1 5CC01F57
 P 7750 1450
-F 0 "#PWR?" H 7750 1300 50  0001 C CNN
+F 0 "#PWR09" H 7750 1300 50  0001 C CNN
 F 1 "+3.3V" H 7750 1590 50  0000 C CNN
 F 2 "" H 7750 1450 50  0000 C CNN
@@
 	7750 1450 8300 1450
 NoConn ~ 9000 1550
+$Comp
+L Connector:Conn_Coaxial J3
+U 1 1 5CBDB00B
+P 7900 1750
+F 0 "J3" H 8000 1634 50  0000 L CNN
+F 1 "Conn_Coaxial" H 8000 1725 50  0000 L CNN
+F 2 "footprints:5227161-1" H 7900 1750 50  0001 C CNN
+F 3 " ~" H 7900 1750 50  0001 C CNN
+	1    7900 1750
+	-1   0    0    1
+$EndComp
+Wire Wire Line
+	8300 1550 7900 1550
+Wire Wire Line
+	8300 1650 8300 1750
+Wire Wire Line
+	8300 1750 8100 1750
+Text Notes 7650 1950 0    50   ~ 0
+50 Ohm BNC
 $EndSCHEMATC

Commit message: NO BNC! YASSS
Parts:
- removed J3: Conn_Coaxial, footprints:5227161-1, symbol Connector:Conn_Coaxial
- removed R1: 10k, Resistor_SMD:R_0805_2012Metric, symbol Device:R
- added J3: Conn_01x02_Male, Connector_Wire:SolderWirePad_1x02_P3.81mm_Drill0.8mm, symbol Connector:Conn_01x02_Male
Connections:
- wire segments 125 -> 132
- no-connect marks 35 -> 36
Other:
- note added: "The translation byte is set by \nxorh and xorl according to \nthe datasheet pg. 9. This layout\nsets it to 0x0F. Sample conversion\nshown below."
- note removed: "50 Ohm BNC"
- note removed: "The translation byte is set by \nxorh and xorl according to \nthe datasheet pg. 9. This layout\nsets it to 0xF. Sample conversion\nshown below."
Changed lines of the file:
@@
 Connection ~ 2350 4100
-$Comp
-L ROVPCB-rescue:+3.3V-power-ROVPCB-rescue-ROVPCB-rescue #PWR0104
-U 1 1 5CB71953
-P 1000 4800
-F 0 "#PWR0104" H 1000 4650 50  0001 C CNN
-F 1 "+3.3V" H 1000 4940 50  0000 C CNN
-F 2 "" H 1000 4800 50  0000 C CNN
-F 3 "" H 1000 4800 50  0000 C CNN
-	1    1000 4800
-	1    0    0    -1
-$EndComp
 $Comp
 L ROVPCB-rescue:GND-power-ROVPCB-rescue-ROVPCB-rescue #PWR0106
@@
 Wire Wire Line
 	3100 1000 3100 1100
-$Comp
-L Device:R R1
-U 1 1 5CBD8F78
-P 1000 4950
-F 0 "R1" H 930 4904 50  0000 R CNN
-F 1 "10k" H 930 4995 50  0000 R CNN
-F 2 "Resistor_SMD:R_0805_2012Metric" V 930 4950 50  0001 C CNN
-F 3 "~" H 1000 4950 50  0001 C CNN
-	1    1000 4950
-	-1   0    0    1
-$EndComp
 Wire Wire Line
 	1000 5100 1750 5100
@@
 Connection ~ 9200 5350
 Wire Wire Line
-	9200 5350 9050 5350
+	9200 5350 9150 5350
 Wire Wire Line
 	9050 5650 9150 5650
@@
 SDAIN: 0x67 --> Translation Byte: 0xF --> SDAOUT: 0x76
 Text Notes 9550 5700 0    50   ~ 0
-The translation byte is set by \nxorh and xorl according to \nthe datasheet pg. 9. This layout\nsets it to 0xF. Sample conversion\nshown below.
+The translation byte is set by \nxorh and xorl according to \nthe datasheet pg. 9. This layout\nsets it to 0x0F. Sample conversion\nshown below.
 Text Notes 4400 4150 0    50   ~ 0
 Default I2C address: 0x77 (SDO--Vdd), 0x76 (SDO--GND)
@@
 	7750 1450 8300 1450
 NoConn ~ 9000 1550
-$Comp
-L Connector:Conn_Coaxial J3
-U 1 1 5CBDB00B
-P 7900 1750
-F 0 "J3" H 8000 1634 50  0000 L CNN
-F 1 "Conn_Coaxial" H 8000 1725 50  0000 L CNN
-F 2 "footprints:5227161-1" H 7900 1750 50  0001 C CNN
-F 3 " ~" H 7900 1750 50  0001 C CNN
-	1    7900 1750
-	-1   0    0    1
-$EndComp
 Wire Wire Line
 	8300 1550 7900 1550
@@
 Wire Wire Line
 	8300 1750 8100 1750
-Text Notes 7650 1950 0    50   ~ 0
-50 Ohm BNC
+$Comp
+L ROVPCB-rescue:GND-power-ROVPCB-rescue-ROVPCB-rescue #PWR011
+U 1 1 5CBE8F10
+P 1000 5100
+F 0 "#PWR011" H 1000 4850 50  0001 C CNN
+F 1 "GND" H 1000 4950 50  0000 C CNN
+F 2 "" H 1000 5100 50  0000 C CNN
+F 3 "" H 1000 5100 50  0000 C CNN
+	1    1000 5100
+	1    0    0    -1
+$EndComp
+$Comp
+L Connector:Conn_01x02_Male J3
+U 1 1 5CBED62E
+P 7500 1750
+F 0 "J3" H 7606 1928 50  0000 C CNN
+F 1 "Conn_01x02_Male" H 7606 1837 50  0000 C CNN
+F 2 "Connector_Wire:SolderWirePad_1x02_P3.81mm_Drill0.8mm" H 7500 1750 50  0001 C CNN
+F 3 "~" H 7500 1750 50  0001 C CNN
+	1    7500 1750
+	1    0    0    -1
+$EndComp
+Wire Wire Line
+	7900 1550 7900 1750
+Wire Wire Line
+	7900 1750 7700 1750
+Wire Wire Line
+	8100 1750 8100 1850
+Wire Wire Line
+	8100 1850 7700 1850
+Wire Wire Line
+	9050 5250 9150 5250
+Wire Wire Line
+	9150 5250 9150 5350
+Connection ~ 9150 5350
+Wire Wire Line
+	9150 5350 9050 5350
+NoConn ~ 7500 5150
 $EndSCHEMATC

Commit message: Pullup resistors in between translater and humidity sensor
Parts:
- added R1, R2: 3k, Resistor_SMD:R_0805_2012Metric, symbol Device:R
Connections:
- net +3V3: now also R1.1, R2.1
- net at U2.3 (SDI), U4.8 (SDAOUT): now also R2.2
- net at U2.4 (SCK), U4.9 (SCLOUT): now also R1.2
Changed lines of the file:
@@
 	7500 5650 7500 6000
 Wire Wire Line
-	7500 5350 6300 5350
+	7500 5350 6800 5350
 Wire Wire Line
 	6300 5350 6300 5450
@@
 	6300 5450 5900 5450
 Wire Wire Line
-	5900 5250 6750 5250
+	5900 5250 6450 5250
 Wire Wire Line
 	6750 5250 6750 5450
@@
 	9150 5350 9050 5350
 NoConn ~ 7500 5150
+$Comp
+L Device:R R1
+U 1 1 5CBE7790
+P 6450 4800
+F 0 "R1" H 6520 4846 50  0000 L CNN
+F 1 "3k" H 6520 4755 50  0000 L CNN
+F 2 "Resistor_SMD:R_0805_2012Metric" V 6380 4800 50  0001 C CNN
+F 3 "~" H 6450 4800 50  0001 C CNN
+	1    6450 4800
+	1    0    0    -1
+$EndComp
+$Comp
+L Device:R R2
+U 1 1 5CBE77D8
+P 6800 4800
+F 0 "R2" H 6870 4846 50  0000 L CNN
+F 1 "3k" H 6870 4755 50  0000 L CNN
+F 2 "Resistor_SMD:R_0805_2012Metric" V 6730 4800 50  0001 C CNN
+F 3 "~" H 6800 4800 50  0001 C CNN
+	1    6800 4800
+	1    0    0    -1
+$EndComp
+Wire Wire Line
+	6450 5250 6450 4950
+Connection ~ 6450 5250
+Wire Wire Line
+	6450 5250 6750 5250
+Wire Wire Line
+	6450 4650 6450 4550
+Wire Wire Line
+	6450 4550 5300 4550
+Wire Wire Line
+	6800 4650 6800 4550
+Wire Wire Line
+	6800 4550 6450 4550
+Connection ~ 6450 4550
+Wire Wire Line
+	6800 4950 6800 5350
+Connection ~ 6800 5350
+Wire Wire Line
+	6800 5350 6300 5350
 $EndSCHEMATC

Commit message: I dont have time
Parts:
- added C4: 10uF, Capacitor_SMD:C_0603_1608Metric, symbol Device:C
- added C5, C6: 0.1uF, Capacitor_SMD:C_0603_1608Metric, symbol Device:C
- added J4: Conn_01x01_Male, Connector_Wire:SolderWirePad_1x01_Drill0.8mm, symbol Connector:Conn_01x01_Male
- added R3: 1k, Resistor_SMD:R_0805_2012Metric, symbol Device:R
- added U6: LTC2451CTS8-TRMPBF, footprints:LTC2451CTS8-TRMPBF, symbol Adafruit_TSL2591-eagle-import:LTC2451CTS8-TRMPBF
- J1, J2: manf# (none) -> DF13-04P-1.25DSA
- P1: manf# (none) -> M52-5001045
- U1: manf# (none) -> MPU-9250
- U2: manf# (none) -> BME280
- U3: manf# (none) -> DFN6_TAOS
- U4: manf# (none) -> LTC4316IDD
- U5: manf# (none) -> EC-OEM
Connections:
- net +3V3: now also U5.9 (NC), C4.1, C5.1, U6.3 (REF+), U6.4 (VCC); no longer U5.3 (Vcc)
- net GND: now also C4.2, C5.2, C6.2, U6.1 (GND), U6.2 (REF-), U6.5 (GND); no longer U5.6 (GND)
- net GPIO2(SDA1): now also U5.7 (INT), U6.8 (SDA); no longer U5.1 (SDA)
- net GPIO3(SCL1): now also U5.2 (NC), U6.7 (SCL); no longer U5.8 (SCL)
- net at U5.10 (NC): now also J3.1 (Pin_1)
- net at U5.4 (PRB-): no longer J3.1 (Pin_1)
- net at U5.5 (PRB+): no longer J3.2 (Pin_2)
- new net: C6.1, R3.2, U6.6 (IN)
- new net: J4.1 (Pin_1), R3.1
Other:
- note added: "ADC for Current Sense"
- moved on the sheet: U5
Changed lines of the file:
@@
 F 2 "Connector_PinSocket_2.54mm:PinSocket_2x20_P2.54mm_Vertical" H -2250 1050 50  0001 C CNN
 F 3 "" H -2250 1050 50  0001 C CNN
+F 4 "M52-5001045" H 2600 2000 50  0001 C CNN "manf#"
 	1    2600 2000
 	1    0    0    -1
@@
 F 2 "Connector_Hirose:Hirose_DF13-04P-1.25DSA_1x04_P1.25mm_Vertical" H 4750 1500 50  0001 C CNN
 F 3 "~" H 4750 1500 50  0001 C CNN
+F 4 "DF13-04P-1.25DSA" H 4750 1500 50  0001 C CNN "manf#"
 	1    4750 1500
 	1    0    0    -1
@@
 F 2 "Connector_Hirose:Hirose_DF13-04P-1.25DSA_1x04_P1.25mm_Vertical" H 4750 2000 50  0001 C CNN
 F 3 "~" H 4750 2000 50  0001 C CNN
+F 4 "DF13-04P-1.25DSA" H 4750 2000 50  0001 C CNN "manf#"
 	1    4750 2000
 	1    0    0    -1
@@
 F 1 "MPU-9250" H 2450 4223 50  0000 C CNN
 F 2 "Sensor_Motion:InvenSense_QFN-24_3x3mm_P0.4mm" H 2450 4300 50  0001 C CNN
-F 3 "https://store.invensense.com/datasheets/invensense/MPU9250REV1.0.pdf" H 2450 5150 50  0001 C CNN
+F 3 "${KIPRJMOD}\\Datasheets\\MPU9250.pdf" H 2450 5150 50  0001 C CNN
+F 4 "MPU-9250" H 2450 5300 50  0001 C CNN "manf#"
 	1    2450 5300
 	1    0    0    -1
@@
 $EndComp
 Wire Wire Line
-	3150 5700 3350 5700
+	3150 5700 3250 5700
 Wire Wire Line
 	2350 4100 1600 4100
@@
 F 1 "BME280" H 4870 5305 50  0000 R CNN
 F 2 "Package_LGA:Bosch_LGA-8_2.5x2.5mm_P0.65mm_ClockwisePinNumbering" H 5300 5150 50  0001 C CNN
-F 3 "https://cdn-shop.adafruit.com/datasheets/BST-BME280_DS001-10.pdf" H 5300 5150 50  0001 C CNN
+F 3 "${KIPRJMOD}\\Datasheets\\BME280.pdf" H 5300 5150 50  0001 C CNN
+F 4 "BME280" H 5300 5350 50  0001 C CNN "manf#"
 	1    5300 5350
 	1    0    0    -1
@@
 F 1 "LIGHT_TSL2591" H 5377 6961 42  0000 L CNN
 F 2 "Adafruit TSL2591:DFN6_TAOS" H 5150 7050 50  0001 C CNN
-F 3 "" H 5150 7050 50  0001 C CNN
+F 3 "${KIPRJMOD}\\Datasheets\\TSL25911.pdf" H 5150 7050 50  0001 C CNN
+F 4 "DFN6_TAOS" H 5150 7050 50  0001 C CNN "manf#"
 	1    5150 7050
 	1    0    0    -1
@@
 F 1 "LTC4316IDDPBF" H 11525 5924 50  0000 C CNN
 F 2 "LTC4316IDDPBF:DFN-10_DD" H 13450 5150 50  0001 L BNN
-F 3 "https://www.analog.com/media/en/technical-documentation/data-sheets/4316fa.pdf" H 13250 5650 50  0001 L BNN
+F 3 "${KIPRJMOD}\\Datasheets\\LTC4316.pdf" H 13250 5650 50  0001 L BNN
 F 4 "Linear Technology/Analog" H 13100 5950 50  0001 L BNN "Field4"
 F 5 "LTC4316 - Single I2C/SMBus Address Translator" H 12700 5800 50  0001 L BNN "Field5"
 F 6 "LTC4316IDD#PBF" H 13350 5300 50  0001 L BNN "Field7"
 F 7 "DFN-10 Linear Technology" H 13150 5500 50  0001 L BNN "Field8"
+F 8 "LTC4316IDD" H 9900 5650 50  0001 C CNN "manf#"
 	1    9900 5650
 	-1   0    0    1
@@
 F 1 "AtlasOEM" H 8650 1684 50  0000 C CNN
 F 2 "Adafruit TSL2591:OEM Board" H 8650 1400 50  0001 C CNN
-F 3 "https://www.atlas-scientific.com/_files/_datasheets/_oem/EC_oem_datasheet.pdf" H 8650 1400 50  0001 C CNN
+F 3 "${KIPRJMOD}\\Datasheets\\EC_oem_datasheet.pdf" H 8650 1400 50  0001 C CNN
+F 4 "EC-OEM" H 8650 1400 50  0001 C CNN "manf#"
 	1    8650 1400
-	1    0    0    -1
+	-1   0    0    1
 $EndComp
 NoConn ~ 9000 1250
@@
 Wire Wire Line
 	6800 5350 6300 5350
+$Comp
+L power:PWR_FLAG #FLG0103
+U 1 1 5CBFE387
+P 3250 5700
+F 0 "#FLG0103" H 3250 5775 50  0001 C CNN
+F 1 "PWR_FLAG" V 3250 5828 50  0000 L CNN
+F 2 "" H 3250 5700 50  0001 C CNN
+F 3 "~" H 3250 5700 50  0001 C CNN
+	1    3250 5700
+	-1   0    0    1
+$EndComp
+Connection ~ 3250 5700
+Wire Wire Line
+	3250 5700 3350 5700
+$Comp
+L Adafruit_TSL2591-eagle-import:LTC2451CTS8-TRMPBF U6
+U 1 1 5CC0994E
+P 7600 2850
+F 0 "U6" H 8825 3237 60  0000 C CNN
+F 1 "LTC2451CTS8-TRMPBF" H 8825 3131 60  0000 C CNN
+F 2 "footprints:LTC2451CTS8-TRMPBF" H 8850 3050 60  0001 C CNN
+F 3 "${KIPRJMOD}\\Datasheets\\LTC2451.pdf" H 8825 3131 60  0001 C CNN
+	1    7600 2850
+	1    0    0    -1
+$EndComp
+Text Label 10150 2950 2    50   ~ 0
+GPIO3(SCL1)
+Text Label 10150 2850 2    50   ~ 0
+GPIO2(SDA1)
+Wire Wire Line
+	9500 2950 10150 2950
+Wire Wire Line
+	10150 2850 9500 2850
+$Comp
+L ROVPCB-rescue:GND-power-ROVPCB-rescue-ROVPCB-rescue #PWR0104
+U 1 1 5CC19AEF
+P 9750 3400
+F 0 "#PWR0104" H 9750 3150 50  0001 C CNN
+F 1 "GND" H 9750 3250 50  0000 C CNN
+F 2 "" H 9750 3400 50  0000 C CNN
+F 3 "" H 9750 3400 50  0000 C CNN
+	1    9750 3400
+	1    0    0    -1
+$EndComp
+$Comp
+L ROVPCB-rescue:GND-power-ROVPCB-rescue-ROVPCB-rescue #PWR0115
+U 1 1 5CC19B4E
+P 7900 2850
+F 0 "#PWR0115" H 7900 2600 50  0001 C CNN
+F 1 "GND" H 7900 2700 50  0000 C CNN
+F 2 "" H 7900 2850 50  0000 C CNN
+F 3 "" H 7900 2850 50  0000 C CNN
+	1    7900 2850
+	1    0    0    -1
+$EndComp
+Wire Wire Line
+	8150 2850 7900 2850
+$Comp
+L ROVPCB-rescue:+3.3V-power-ROVPCB-rescue-ROVPCB-rescue #PWR0116
+U 1 1 5CC1F2DC
+P 7650 3150
+F 0 "#PWR0116" H 7650 3000 50  0001 C CNN
+F 1 "+3.3V" H 7650 3290 50  0000 C CNN
+F 2 "" H 7650 3150 50  0000 C CNN
+F 3 "" H 7650 3150 50  0000 C CNN
+	1    7650 3150
+	1    0    0    -1
+$EndComp
+$Comp
+L Device:C C5
+U 1 1 5CC24DAB
+P 8050 3400
+F 0 "C5" H 8165 3446 50  0000 L CNN
+F 1 "0.1uF" H 8165 3355 50  0000 L CNN
+F 2 "Capacitor_SMD:C_0603_1608Metric" H 8088 3250 50  0001 C CNN
+F 3 "~" H 8050 3400 50  0001 C CNN
+	1    8050 3400
+	1    0    0    -1
+$EndComp
+Wire Wire Line
+	8150 2850 8150 2950
+Connection ~ 8150 2850
+$Comp
+L Device:C C4
+U 1 1 5CC2A628
+P 7650 3400
+F 0 "C4" H 7765 3446 50  0000 L CNN
+F 1 "10uF" H 7765 3355 50  0000 L CNN
+F 2 "Capacitor_SMD:C_0603_1608Metric" H 7688 3250 50  0001 C CNN
+F 3 "~" H 7650 3400 50  0001 C CNN
+	1    7650 3400
+	1    0    0    -1
+$EndComp
+Wire Wire Line
+	7650 3150 7650 3250
+Wire Wire Line
+	8150 3150 8050 3150
+Connection ~ 7650 3150
+Wire Wire Line
+	8050 3150 8050 3250
+Connection ~ 8050 3150
+Wire Wire Line
+	8050 3150 7650 3150
+Wire Wire Line
+	8150 3050 8150 3150
+Connection ~ 8150 3150
+$Comp
+L ROVPCB-rescue:GND-power-ROVPCB-rescue-ROVPCB-rescue #PWR0117
+U 1 1 5CC40D88
+P 8050 3550
+F 0 "#PWR0117" H 8050 3300 50  0001 C CNN
+F 1 "GND" H 8050 3400 50  0000 C CNN
+F 2 "" H 8050 3550 50  0000 C CNN
+F 3 "" H 8050 3550 50  0000 C CNN
+	1    8050 3550
+	1    0    0    -1
+$EndComp
+$Comp
+L ROVPCB-rescue:GND-power-ROVPCB-rescue-ROVPCB-rescue #PWR0118
+U 1 1 5CC46ADC
+P 7650 3550
+F 0 "#PWR0118" H 7650 3300 50  0001 C CNN
+F 1 "GND" H 7650 3400 50  0000 C CNN
+F 2 "" H 7650 3550 50  0000 C CNN
+F 3 "" H 7650 3550 50  0000 C CNN
+	1    7650 3550
+	1    0    0    -1
+$EndComp
+Text Notes 7550 2350 0    138  ~ 28
+ADC for Current Sense
+Wire Wire Line
+	9550 3150 9500 3150
+$Comp
+L Device:C C6
+U 1 1 5CC5F4A9
+P 9750 3200
+F 0 "C6" H 9865 3246 50  0000 L CNN
+F 1 "0.1uF" H 9865 3155 50  0000 L CNN
+F 2 "Capacitor_SMD:C_0603_1608Metric" H 9788 3050 50  0001 C CNN
+F 3 "~" H 9750 3200 50  0001 C CNN
+	1    9750 3200
+	1    0    0    -1
+$EndComp
+Wire Wire Line
+	9750 3350 9750 3400
+Wire Wire Line
+	9550 3150 9550 3350
+Wire Wire Line
+	9550 3350 9750 3350
+Connection ~ 9750 3350
+Wire Wire Line
+	9750 3050 9500 3050
+$Comp
+L Device:R R3
+U 1 1 5CC715CB
+P 10250 3050
+F 0 "R3" H 10320 3096 50  0000 L CNN
+F 1 "1k" H 10320 3005 50  0000 L CNN
+F 2 "Resistor_SMD:R_0805_2012Metric" V 10180 3050 50  0001 C CNN
+F 3 "~" H 10250 3050 50  0001 C CNN
+	1    10250 3050
+	0    1    1    0
+$EndComp
+Wire Wire Line
+	10100 3050 9750 3050
+Connection ~ 9750 3050
+$Comp
+L Connector:Conn_01x01_Male J4
+U 1 1 5CC779A0
+P 10700 3050
+F 0 "J4" H 10700 3150 50  0000 R CNN
+F 1 "Conn_01x01_Male" H 10900 3250 50  0000 R CNN
+F 2 "Connector_Wire:SolderWirePad_1x01_Drill0.8mm" H 10700 3050 50  0001 C CNN
+F 3 "~" H 10700 3050 50  0001 C CNN
+	1    10700 3050
+	-1   0    0    1
+$EndComp
+Wire Wire Line
+	10500 3050 10400 3050
 $EndSCHEMATC

Commit message: Fixed DRC errors and other things
Connections:
- net +3V3: now also U5.3 (Vcc); no longer U5.9 (NC)
- net GND: now also U5.6 (GND)
- net GPIO2(SDA1): now also U5.1 (SDA); no longer U5.7 (INT)
- net GPIO3(SCL1): now also U5.8 (SCL); no longer U5.2 (NC)
- net at U5.10 (NC): no longer J3.1 (Pin_1)
- net at U5.4 (PRB-): now also J3.1 (Pin_1)
- net at U5.5 (PRB+): now also J3.2 (Pin_2)
Other:
- moved on the sheet: U5
Changed lines of the file:
@@
 	3000 2000 3000 2500
-Wire Wire Line
-	2300 3000 2300 3150
 Wire Wire Line
 	2200 1100 2200 1900
@@
 $EndComp
 Wire Wire Line
-	3150 5700 3250 5700
-Wire Wire Line
 	2350 4100 1600 4100
 Wire Wire Line
@@
 Wire Wire Line
 	5300 4550 5300 4650
-Wire Wire Line
-	6200 4900 5900 4900
 Wire Wire Line
 	5900 4900 5900 5050
@@
 F 4 "EC-OEM" H 8650 1400 50  0001 C CNN "manf#"
 	1    8650 1400
-	-1   0    0    1
+	1    0    0    -1
 $EndComp
 NoConn ~ 9000 1250
@@
 Wire Wire Line
 	6800 5350 6300 5350
-$Comp
-L power:PWR_FLAG #FLG0103
-U 1 1 5CBFE387
-P 3250 5700
-F 0 "#FLG0103" H 3250 5775 50  0001 C CNN
-F 1 "PWR_FLAG" V 3250 5828 50  0000 L CNN
-F 2 "" H 3250 5700 50  0001 C CNN
-F 3 "~" H 3250 5700 50  0001 C CNN
-	1    3250 5700
-	-1   0    0    1
-$EndComp
-Connection ~ 3250 5700
-Wire Wire Line
-	3250 5700 3350 5700
 $Comp
 L Adafruit_TSL2591-eagle-import:LTC2451CTS8-TRMPBF U6
@@
 Wire Wire Line
 	10500 3050 10400 3050
+Wire Wire Line
+	3150 5700 3350 5700
+Wire Wire Line
+	5900 4900 6200 4900
+Wire Wire Line
+	2300 3000 2300 3150
 $EndSCHEMATC

Commit message: I think it is done!
Parts:
- U4: footprint LTC4316IDDPBF:DFN-10_DD -> Package_SO:MSOP-10_3x3mm_P0.5mm
Changed lines of the file:
@@
 F 0 "U4" H 11525 6015 50  0000 C CNN
 F 1 "LTC4316IDDPBF" H 11525 5924 50  0000 C CNN
-F 2 "LTC4316IDDPBF:DFN-10_DD" H 13450 5150 50  0001 L BNN
+F 2 "Package_SO:MSOP-10_3x3mm_P0.5mm" H 13450 5150 50  0001 L BNN
 F 3 "${KIPRJMOD}\\Datasheets\\LTC4316.pdf" H 13250 5650 50  0001 L BNN
 F 4 "Linear Technology/Analog" H 13100 5950 50  0001 L BNN "Field4"
